File: Test.kicad_pcb (KiCad board)
At the start: 4 copper layers, 123.5 x 73 mm, 20 parts, among them J1 AVR-ISP-6, P1 USB_C_Receptacle_USB2.0, SW1 SW_Push, U1 ATmega328P-P, U2 CH340N, U3 AMS1117, Y1 Crystal

Commit message: Update Test.kicad_pcb
Parts:
- DS1: value HY1602E -> WC1602A; footprint Display:HY1602E -> Display:WC1602A
- moved DS1 25.9 mm to (123.8, 105.1)
- moved R2 6.08 mm to (161.0, 101.0)
- moved R6 0.51 mm to (171.5, 92.5)
Connections:
- DS1 pad 11: unconnected-(DS1-DB2-Pad11) -> Net-(DS1-D4)
- DS1 pad 12: unconnected-(DS1-DB3-Pad12) -> Net-(DS1-D5)
- DS1 pad 13: Net-(DS1-DB4) -> Net-(DS1-D6)
- DS1 pad 14: Net-(DS1-DB5) -> Net-(DS1-D7)
- DS1 pad 15: Net-(DS1-DB6) -> unconnected-(DS1-LED(+)-Pad15)
- DS1 pad 16: Net-(DS1-DB7) -> Net-(DS1-LED(-))
- DS1 pad 2: Net-(DS1-LEDA) -> +5V
- DS1 pad 3: GND -> Net-(DS1-VO)
- DS1 pad 4: +5V -> Net-(DS1-RS)
- DS1 pad 5: Net-(DS1-Vo) -> GND
- DS1 pad 6: Net-(DS1-RS) -> Net-(DS1-E)
- DS1 pad 7: GND -> unconnected-(DS1-D0-Pad7)
- R2 pad 1: Net-(DS1-LEDA) -> GND
- R2 pad 2: +5V -> Net-(DS1-LED(-))
- R3 pad 2: Net-(DS1-Vo) -> Net-(DS1-VO)
- U1 pad 11: Net-(DS1-DB5) -> Net-(DS1-D5)
- U1 pad 12: Net-(DS1-DB6) -> Net-(DS1-D6)
- U1 pad 13: Net-(DS1-DB7) -> Net-(DS1-D7)
- U1 pad 5: unconnected-(U1-PD3-Pad5) -> Net-(DS1-E)
- U1 pad 6: Net-(DS1-DB4) -> Net-(DS1-D4)
Routing:
- net Net-(DS1-D7): track 0.00 -> 47.1 mm
- net Net-(DS1-D6): track 0.00 -> 46.8 mm
- net Net-(DS1-D5): track 0.00 -> 46.5 mm
- net Net-(DS1-E): track 0.00 -> 45.0 mm
- net Net-(DS1-D4): track 0.00 -> 37.3 mm
- net Net-(DS1-VO): track 0.00 -> 33.5 mm
- net Net-(DS1-RS): track 16.9 -> 50.2 mm, vias 0 -> 2
- net Net-(DS1-DB7): track 15.8 -> 0.00 mm
- net Net-(DS1-DB6): track 15.8 -> 0.00 mm
- net Net-(DS1-DB5): track 15.8 -> 0.00 mm
- net Net-(DS1-DB4): track 14.6 -> 0.00 mm
- net Net-(DS1-Vo): track 5.69 -> 0.00 mm
- net Net-(DS1-LEDA): track 5.47 -> 0.00 mm
- net +5V: track 35.6 -> 31.5 mm
- net Net-(DS1-LED(-)): track 0.00 -> 4.08 mm

Commit message: Update Test.kicad_pcb
Parts:
- P1: footprint Connector_USB:USB_C_Receptacle_GCT_USB4085 -> Connector_USB:USB_C_Receptacle_GCT_USB4105-xx-A_16P_TopMnt_Horizontal
- moved P1 4.36 mm to (167.0, 69.4)
Routing:
- net GND: track 0.00 -> 2.72 mm
- net USB_C D+: track 4.72 -> 2.40 mm
- net Net-(P1-CC2): track 8.32 -> 10.5 mm, vias 0 -> 1
- net Net-(U3-VI): track 14.1 -> 12.2 mm
- net USB_C D-: track 4.20 -> 4.90 mm
- net Net-(P1-CC1): track 4.68 -> 4.39 mm, vias 0 -> 1

Commit message: Caleb's changes
Parts:
- moved G*** 21.7 mm to (109.5, 100.5)
- moved C1 16.4 mm to (161.5, 86.5)
- moved C2 16.4 mm to (170.0, 82.0)
- moved D1 16.4 mm to (113.4, 90.0)
- moved D2 16.4 mm to (118.9, 90.0)
- moved DS1 16.4 mm to (109.8, 113.6)
- moved J1 16.4 mm to (178.5, 78.4)
- moved P1 16.4 mm to (153.0, 77.9)
- moved R1 16.4 mm to (135.5, 97.0)
- moved R2 16.4 mm to (147.0, 109.5)
- moved R3 16.4 mm to (140.0, 97.0)
- moved R4 16.4 mm to (157.0, 85.5)
- moved R5 16.4 mm to (144.0, 77.6)
- moved R6 16.4 mm to (157.5, 101.0)
- moved R7 16.4 mm to (152.1, 101.0)
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Other:
- board size 123.5 x 73 mm -> 85 x 75 mm
